Commit message: Updated gazebo_ur5e.xacro to include a physical camera link and a dedicated optical frame aligned with REP-103 standards. Configured the libgazebo_ros_camera.so plugin and the gz-sim-sensors-system to enable real-time image rendering.

File: src/ur5e_xbox_joint_publisher/urdf/gazebo_ur5e.xacro (robot description, xacro)
@@ -33,3 +33,50 @@
      </plugin>
    </gazebo>
+   <link name="camera_link">
+    <visual>
+      <geometry><box size="0.02 0.05 0.02"/></geometry>
+      <material name="black"><color rgba="0 0 0 1"/></material>
+    </visual>
+  </link>
+  <link name="camera_link_optical"/>
+  <joint name="camera_optical_joint" type="fixed">
+    <origin xyz="0 0 0" rpy="-1.5708 0 -1.5708"/>
+    <parent link="camera_link"/>
+    <child link="camera_link_optical"/>
+  </joint>
+  <joint name="camera_joint" type="fixed">
+    <parent link="tool0"/>
+    <child link="camera_link"/>
+    <origin xyz="0 0 0.02" rpy="1.5708 -1.5708 0"/>
+  </joint>
+  <gazebo reference="camera_link">
+    <sensor name="ur5e_camera" type="camera">
+      <camera>
+        <horizontal_fov>1.089</horizontal_fov>
+        <image>
+          <width>640</width>
+          <height>480</height>
+          <format>R8G8B8</format>
+        </image>
+        <clip>
+          <near>0.05</near>
+          <far>8.0</far>
+        </clip>
+      </camera>
+      <always_on>1</always_on>
+      <update_rate>30</update_rate>
+      <visualize>true</visualize>
+      <topic>camera/image_raw</topic>
+      <plugin name="camera_controller" filename="libgazebo_ros_camera.so">
+        <frame_name>camera_link</frame_name>
+      </plugin>
+    </sensor>
+  </gazebo>
+  <gazebo>
+    <plugin
+      filename="gz-sim-sensors-system"
+      name="gz::sim::systems::Sensors">
+      <render_engine>ogre2</render_engine>
+    </plugin>
+  </gazebo>
 </robot>

Commit message: feat: integrate Robotiq 2F-85 gripper and mimic joint plugins
- Included Robotiq description macro and attached to tool0.
- Added gripper joints to ros2_control GazeboSimSystem.
- Configured gz-sim-joint-mimic-system plugins for parallel gripper linkage.
- Relocated camera_joint to robotiq_85_base_link for better visibility.
- Defined surface friction (mu1/mu2) for gripper fingertips.

File: src/ur5e_xbox_joint_publisher/urdf/gazebo_ur5e.xacro (robot description, xacro)
@@ -1,37 +1,50 @@
 <?xml version="1.0"?>
 <robot xmlns:xacro="http://wiki.ros.org/xacro" name="ur5e">
-   <xacro:arg name="name" default="ur"/>
-   <xacro:arg name="ur_type" default="ur5e"/>
-   <xacro:arg name="tf_prefix" default="" />
-   <xacro:include filename="$(find ur_description)/urdf/ur_macro.xacro"/>
-   <link name="world" />
-   <xacro:ur_robot
-     name="$(arg name)"
-     tf_prefix="$(arg tf_prefix)"
-     parent="world"
-     joint_limits_parameters_file="$(find ur_description)/config/$(arg ur_type)/joint_limits.yaml"
-     kinematics_parameters_file="$(find ur_description)/config/$(arg ur_type)/default_kinematics.yaml"
-     physical_parameters_file="$(find ur_description)/config/$(arg ur_type)/physical_parameters.yaml"
-     visual_parameters_file="$(find ur_description)/config/$(arg ur_type)/visual_parameters.yaml"
-     >
-     <origin xyz="0 0 0" rpy="0 0 0" />
-   </xacro:ur_robot>
-   <ros2_control name="GazeboSimSystem" type="system">
-     <hardware>
-       <plugin>gz_ros2_control/GazeboSimSystem</plugin>
-     </hardware>
-     <joint name="shoulder_pan_joint"><command_interface name="position"/><state_interface name="position"/><state_interface name="velocity"/></joint>
-     <joint name="shoulder_lift_joint"><command_interface name="position"/><state_interface name="position"/><state_interface name="velocity"/></joint>
-     <joint name="elbow_joint"><command_interface name="position"/><state_interface name="position"/><state_interface name="velocity"/></joint>
-     <joint name="wrist_1_joint"><command_interface name="position"/><state_interface name="position"/><state_interface name="velocity"/></joint>
-     <joint name="wrist_2_joint"><command_interface name="position"/><state_interface name="position"/><state_interface name="velocity"/></joint>
-     <joint name="wrist_3_joint"><command_interface name="position"/><state_interface name="position"/><state_interface name="velocity"/></joint>
-   </ros2_control>
-   <gazebo>
-     <plugin filename="gz_ros2_control-system" name="gz_ros2_control::GazeboSimROS2ControlPlugin">
-       <parameters>$(find ur5e_xbox_joint_publisher)/config/ur5e_controllers.yaml</parameters>
-     </plugin>
-   </gazebo>
-   <link name="camera_link">
+  <xacro:arg name="name" default="ur"/>
+  <xacro:arg name="ur_type" default="ur5e"/>
+  <xacro:arg name="tf_prefix" default="" />
+  <xacro:include filename="$(find ur_description)/urdf/ur_macro.xacro"/>
+  <xacro:include filename="$(find robotiq_description)/urdf/robotiq_2f_85_macro.urdf.xacro" />
+  <link name="world" />
+  <xacro:ur_robot
+    name="$(arg name)"
+    tf_prefix="$(arg tf_prefix)"
+    parent="world"
+    joint_limits_parameters_file="$(find ur_description)/config/$(arg ur_type)/joint_limits.yaml"
+    kinematics_parameters_file="$(find ur_description)/config/$(arg ur_type)/default_kinematics.yaml"
+    physical_parameters_file="$(find ur_description)/config/$(arg ur_type)/physical_parameters.yaml"
+    visual_parameters_file="$(find ur_description)/config/$(arg ur_type)/visual_parameters.yaml"
+    >
+    <origin xyz="0 0 0" rpy="0 0 0" />
+  </xacro:ur_robot>
+  <xacro:robotiq_gripper
+    name="robotiq_85"
+    prefix=""
+    parent="tool0">
+    <origin xyz="0 0 0" rpy="0 0 0" />
+  </xacro:robotiq_gripper>
+  <ros2_control name="GazeboSimSystem" type="system">
+    <hardware>
+      <plugin>gz_ros2_control/GazeboSimSystem</plugin>
+      <param name="calculate_dynamics">true</param>
+    </hardware>
+    <joint name="shoulder_pan_joint"><command_interface name="position"/><state_interface name="position"/><state_interface name="velocity"/></joint>
+    <joint name="shoulder_lift_joint"><command_interface name="position"/><state_interface name="position"/><state_interface name="velocity"/></joint>
+    <joint name="elbow_joint"><command_interface name="position"/><state_interface name="position"/><state_interface name="velocity"/></joint>
+    <joint name="wrist_1_joint"><command_interface name="position"/><state_interface name="position"/><state_interface name="velocity"/></joint>
+    <joint name="wrist_2_joint"><command_interface name="position"/><state_interface name="position"/><state_interface name="velocity"/></joint>
+    <joint name="wrist_3_joint"><command_interface name="position"/><state_interface name="position"/><state_interface name="velocity"/></joint>
+    <joint name="robotiq_85_left_knuckle_joint">
+      <command_interface name="position"/>
+      <state_interface name="position"><param name="initial_value">0.0</param></state_interface>
+      <state_interface name="velocity"/>
+    </joint>
+    <joint name="robotiq_85_right_knuckle_joint"><state_interface name="position"/><state_interface name="velocity"/></joint>
+    <joint name="robotiq_85_left_inner_knuckle_joint"><state_interface name="position"/><state_interface name="velocity"/></joint>
+    <joint name="robotiq_85_right_inner_knuckle_joint"><state_interface name="position"/><state_interface name="velocity"/></joint>
+    <joint name="robotiq_85_left_finger_tip_joint"><state_interface name="position"/><state_interface name="velocity"/></joint>
+    <joint name="robotiq_85_right_finger_tip_joint"><state_interface name="position"/><state_interface name="velocity"/></joint>
+  </ros2_control>
+  <link name="camera_link">
     <visual>
       <geometry><box size="0.02 0.05 0.02"/></geometry>
@@ -46,21 +59,47 @@
   </joint>
   <joint name="camera_joint" type="fixed">
-    <parent link="tool0"/>
+    <parent link="robotiq_85_base_link"/>
     <child link="camera_link"/>
-    <origin xyz="0 0 0.02" rpy="1.5708 -1.5708 0"/>
+    <origin xyz="0 0.05 0.05" rpy="1.5708 -1.5708 0"/>
   </joint>
+  <gazebo>
+    <plugin filename="gz_ros2_control-system" name="gz_ros2_control::GazeboSimROS2ControlPlugin">
+      <parameters>$(find ur5e_xbox_joint_publisher)/config/ur5e_controllers.yaml</parameters>
+    </plugin>
+    <plugin filename="gz-sim-sensors-system" name="gz::sim::systems::Sensors">
+      <render_engine>ogre2</render_engine>
+    </plugin>
+    <plugin filename="gz-sim-joint-mimic-system" name="gz::sim::systems::JointMimic">
+      <joint_name>robotiq_85_left_knuckle_joint</joint_name>
+      <mimic_joint>robotiq_85_right_knuckle_joint</mimic_joint>
+      <multiplier>1.0</multiplier>
+    </plugin>
+    <plugin filename="gz-sim-joint-mimic-system" name="gz::sim::systems::JointMimic">
+      <joint_name>robotiq_85_left_knuckle_joint</joint_name>
+      <mimic_joint>robotiq_85_left_inner_knuckle_joint</mimic_joint>
+      <multiplier>1.0</multiplier>
+    </plugin>
+    <plugin filename="gz-sim-joint-mimic-system" name="gz::sim::systems::JointMimic">
+      <joint_name>robotiq_85_left_knuckle_joint</joint_name>
+      <mimic_joint>robotiq_85_right_inner_knuckle_joint</mimic_joint>
+      <multiplier>1.0</multiplier>
+    </plugin>
+    <plugin filename="gz-sim-joint-mimic-system" name="gz::sim::systems::JointMimic">
+      <joint_name>robotiq_85_left_knuckle_joint</joint_name>
+      <mimic_joint>robotiq_85_left_finger_tip_joint</mimic_joint>
+      <multiplier>-1.0</multiplier>
+    </plugin>
+    <plugin filename="gz-sim-joint-mimic-system" name="gz::sim::systems::JointMimic">
+      <joint_name>robotiq_85_left_knuckle_joint</joint_name>
+      <mimic_joint>robotiq_85_right_finger_tip_joint</mimic_joint>
+      <multiplier>-1.0</multiplier>
+    </plugin>
+  </gazebo>
   <gazebo reference="camera_link">
     <sensor name="ur5e_camera" type="camera">
       <camera>
         <horizontal_fov>1.089</horizontal_fov>
-        <image>
-          <width>640</width>
-          <height>480</height>
-          <format>R8G8B8</format>
-        </image>
-        <clip>
-          <near>0.05</near>
-          <far>8.0</far>
-        </clip>
+        <image><width>640</width><height>480</height><format>R8G8B8</format></image>
+        <clip><near>0.05</near><far>8.0</far></clip>
       </camera>
       <always_on>1</always_on>
@@ -68,15 +107,23 @@
       <visualize>true</visualize>
       <topic>camera/image_raw</topic>
-      <plugin name="camera_controller" filename="libgazebo_ros_camera.so">
-        <frame_name>camera_link</frame_name>
-      </plugin>
     </sensor>
   </gazebo>
-  <gazebo>
-    <plugin
-      filename="gz-sim-sensors-system"
-      name="gz::sim::systems::Sensors">
-      <render_engine>ogre2</render_engine>
-    </plugin>
+  <gazebo reference="robotiq_85_base_link">
+    <self_collide>false</self_collide>
+  </gazebo>
+  <gazebo reference="robotiq_85_left_knuckle_link">
+    <self_collide>false</self_collide>
+    <mu1>1.1</mu1><mu2>1.1</mu2>
+  </gazebo>
+  <gazebo reference="robotiq_85_right_knuckle_link">
+    <self_collide>false</self_collide>
+    <mu1>1.1</mu1><mu2>1.1</mu2>
+  </gazebo>
+  <gazebo reference="robotiq_85_left_finger_tip_link">
+    <self_collide>false</self_collide>
+    <mu1>1.5</mu1><mu2>1.5</mu2> </gazebo>
+  <gazebo reference="robotiq_85_right_finger_tip_link">
+    <self_collide>false</self_collide>
+    <mu1>1.5</mu1><mu2>1.5</mu2>
   </gazebo>
 </robot>
